File: pcb/Macropad.kicad_pcb (KiCad board)
At the start: 2 copper layers, 65 x 85 mm, 25 parts, among them J1 OLED_128x32, SW1 RotaryEncoder_Switch, SW2 SW_Push_45deg, SW3 SW_Push_45deg, SW4 SW_Push_45deg, SW5 SW_Push_45deg, SW6 SW_Push_45deg, SW7 SW_Push_45deg, SW8 SW_Push_45deg, U1 MCU_Seeed_XIAO_RP2040

Commit message: Fix Rotary Encoder
Connections:
- SW1 pad C: unconnected-(SW1-PadC) -> GND
