File: pcb/Macropad.kicad_sch (KiCad schematic)
At the start: 25 parts, among them J1 OLED_128x32, SW1 RotaryEncoder_Switch, SW2 SW_Push_45deg, SW3 SW_Push_45deg, SW4 SW_Push_45deg, SW5 SW_Push_45deg, SW6 SW_Push_45deg, SW7 SW_Push_45deg, SW8 SW_Push_45deg, U1 MCU_Seeed_XIAO_RP2040

Commit message: Fix Rotary Encoder
Connections:
- net GND: now also SW1.C
Changed lines of the file:
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@@
 		)
 	)
-	(text_box "RGP Matrix"
+	(text_box "RGB Matrix"
 		(exclude_from_sim no)
 		(at 30.48 64.77 0)
@@
 					(unit 1)
 				)
+			)
+		)
+	)
+	(symbol
+		(lib_id "power:GND")
+		(at 149.86 36.83 270)
+		(unit 1)
+		(exclude_from_sim no)
+		(in_bom yes)
+		(on_board yes)
+		(dnp no)
+		(property "Reference" "#PWR010"
+			(at 143.51 36.83 0)
+			(effects
+				(font
+					(size 1.27 1.27)
+				)
+				(hide yes)
+			)
+		)
+		(property "Value" "GND"
+			(at 144.78 36.83 0)
+			(effects
+				(font
+					(size 1.27 1.27)
+				)
+			)
+		)
+		(property "Footprint" ""
+			(at 149.86 36.83 0)
+			(effects
+				(font
+					(size 1.27 1.27)
+				)
+				(hide yes)
+			)
+		)
+		(property "Datasheet" ""
+			(at 149.86 36.83 0)
+			(effects
+				(font
+					(size 1.27 1.27)
+				)
+				(hide yes)
+			)
+		)
+		(property "Description" "Power symbol creates a global label with name \"GND\" , ground"
+			(at 149.86 36.83 0)
+			(effects
+				(font
+					(size 1.27 1.27)
+				)
+				(hide yes)
+			)
+		)
+		(pin "1"
+		)
+		(instances
+			(project "Macropad"
+				(path "/3b46d3fc-ddd1-4fb8-b937-79db70ce81ac"
+					(reference "#PWR010")
+					(unit 1)
+				)
